File: stm-breakout.sch (EAGLE design)
At the start: 5 parts, among them IC1 STM32H757IIT6

Commit message: Add in power filtering and SMPS functionality
Parts:
- added C1, C10, C11, C55, C56, C6, C7, C8, C9: 2.2u, rcl:C-EUC0603
- added C12, C13, C16, C18, C20, C22, C24, C26, C28, C30, C32, C34, C36, C38, C40, C42, C44, C46, C49, C5: 4.7u, rcl:C-EUC0603
- added C14, C17, C19, C2, C21, C23, C25, C27, C29, C3, C31, C33, C35, C37, C39, C41, C43, C45, C47, C48: 100n, rcl:C-EUC0402
- added C15, C4: 1u, rcl:C-EUC0603
- added C50, C52, C53, C54: 10u, rcl:C-EUC0603
- added C51: 220p, rcl:C-EUC0402
- added L1: VLS3015CX-2R2M-H, SamacSys_Parts:VLS3015CX-2R2M-H
Connections:
- new net GND: C1.2, C11.2, C12.2, C13.2, C14.2, C17.2, C19.2, C2.2, C21.2, C23.2, C25.2, C27.2, C29.2, C3.2, C31.2, C33.2, C35.2, C37.2, C39.2, C41.2, C43.2, C45.2, C47.2, C48.2, C49.2, C5.2, C50.2, C51.2, C52.2, C53.2, C54.2, C55.2, C56.2, C7.2, C9.2, IC1.VSSA, IC1.VSSDSI_1, IC1.VSSDSI_2, IC1.VSSSMPS, IC1.VSS_1, IC1.VSS_10, IC1.VSS_11, IC1.VSS_12, IC1.VSS_13, IC1.VSS_14, IC1.VSS_15, IC1.VSS_16, IC1.VSS_17, IC1.VSS_18, IC1.VSS_2, IC1.VSS_3, IC1.VSS_4, IC1.VSS_5, IC1.VSS_6, IC1.VSS_7, IC1.VSS_8, IC1.VSS_9
- new net N$1: C2.1, C4.2
- new net N$2: C6.2, C7.1
- new net N$3: C8.2, C9.1
- new net N$4: C10.2, C11.1
- new net VCAPDSI: C1.1, C55.1, C56.1, IC1.VCAPDSI, IC1.VDD12DSI_1, IC1.VDD12DSI_2
- new net VDD: C10.1, C12.1, C13.1, C16.1, C18.1, C20.1, C22.1, C24.1, C26.1, C28.1, C30.1, C32.1, C34.1, C36.1, C38.1, C4.1, C40.1, C42.1, C44.1, C46.1, C5.1, C50.1, C52.1, C53.1, C54.1, C6.1, C8.1, IC1.VCAP_1, IC1.VCAP_2, IC1.VCAP_3, IC1.VDDA, IC1.VDDLDO_1, IC1.VDDLDO_2, IC1.VDDLDO_3, IC1.VDD_1, IC1.VDD_10, IC1.VDD_11, IC1.VDD_12, IC1.VDD_13, IC1.VDD_14, IC1.VDD_15, IC1.VDD_16, IC1.VDD_2, IC1.VDD_3, IC1.VDD_4, IC1.VDD_5, IC1.VDD_6, IC1.VDD_7, IC1.VDD_8, IC1.VDD_9, IC1.VFBSMPS, L1.1
- new net VDD33USB: C48.1, IC1.VDD33USB
- new net VDD50USB: C47.1, IC1.VDD50USB
- new net VIN: C49.1, IC1.VDDSMPS
- new net VLXSMPS: C51.1, IC1.VLXSMPS, L1.2
- new net VREF: C15.1, IC1.VREF+
- new net VREFNF: C14.1, C15.2
- new net VREFNF1: C16.2, C3.1
- new net VREFNF10: C33.1, C34.2
- new net VREFNF11: C35.1, C36.2
- new net VREFNF12: C37.1, C38.2
- new net VREFNF13: C39.1, C40.2
- new net VREFNF14: C41.1, C42.2
- new net VREFNF15: C43.1, C44.2
- new net VREFNF16: C45.1, C46.2
- new net VREFNF2: C17.1, C18.2
- new net VREFNF3: C19.1, C20.2
- new net VREFNF4: C21.1, C22.2
- new net VREFNF5: C23.1, C24.2
- new net VREFNF6: C25.1, C26.2
- new net VREFNF7: C27.1, C28.2
- new net VREFNF8: C29.1, C30.2
- new net VREFNF9: C31.1, C32.2
Other:
- note added: "From 16 VDD Pins"
- note added: "From 3 VDDldo pins"
- note added: "From 3 Vcap pins"
- note added: "From VSSA"
- note added: "SMPS"
- note added: "USB Regulator"
- note added: "VDDLDO"
- note added: "VFBSMPS"
- note added: "Vcap"
- note added: "Vref"

Commit message: Add nrst switch, sdcard, TFT display connector, and jtag
Parts:
- removed JP1, JP2, JP3, JP4: (no value), pinhead:PINHD-2X22
- added C57: 100n, rcl:C-EUC0402
- added J1: FTSH-107-01-L-DV-K-A, SamacSys_Parts:FTSH-107-01-L-DV-K-A
- added J2: DM3CS-SF, SamacSys_Parts:DM3CS-SF
- added J3: FH12-14S-0.5SH_55_, SamacSys_Parts:FH12-14S-0.5SH_55_
- added JP5: (no value), pinhead:PINHD-1X10
- added JP6: (no value), SamacSys_Parts:JP2
- added R1: 1k, rcl:R-US_R0402
- added S1: B3FS-1000P, SamacSys_Parts:B3FS-1000P
Connections:
- new net BOOT0: IC1.BOOT0, JP6.2
- new net DA: J3.11, R1.2
- new net JCLK: IC1.PA14, J1.6
- new net JTDI: IC1.PA15, J1.10
- new net JTDO: IC1.PB3, J1.8
- new net JTMS: IC1.PA13, J1.4
- new net NRST: C57.1, IC1.NRST, J1.12, J3.8, JP5.4, S1.1, S1.3
- new net RS: IC1.PA6, J3.9
- new net SDMMC1_CK: IC1.PC12, J2.CLK
- new net SDMMC1_CMD: IC1.PD2, J2.CMD
- new net SDMMC1_D0: IC1.PC8, J2.DAT0
- new net SDMMC1_D1: IC1.PC9, J2.DAT1
- new net SDMMC1_D2: IC1.PC10, J2.DAT2
- new net SDMMC1_D3: IC1.PC11, J2.CD/DAT3
- new net SPI1_MOSI: IC1.PA7, R1.1
- new net SPI1_NSS: IC1.PA4, J3.7
- new net SPI1_SCK: IC1.PA5, J3.10
- new net UART4_RX: IC1.PD0, J1.13
- new net UART4_TX: IC1.PD1, J1.14
- new net VBAT: IC1.VBAT, JP5.2
- new net XL: J3.2
- new net XR: J3.4
- new net YD: J3.3
- new net YU: J3.1
- net GND: now also C57.2, IC1.PDR_ON, J1.11, J1.5, J1.7, J1.9, J2.MP1, J2.MP2, J2.MP3, J2.MP4, J2.MP5, J2.VSS, J3.13, J3.5, J3.MP1, J3.MP2, JP5.1, JP6.3, S1.2, S1.4
- net VDD: now also J1.3, J2.VDD, J3.14, J3.6, JP6.1
- net VIN: now also JP5.3
Other:
- note added: "STDC14 for STLinkV3"
